File: electronics/view_base/view_base.kicad_sch (KiCad schematic)
At the start: 107 parts, among them J1 BLDC, J2 USB_C_Receptacle_USB2.0, J3 LCD, J4 A, J5 B, Q1 MMBT4403, Q2 UMH3N, U1 MT6701-CT, U2 T-Micro32_Plus, U3 CH340C, U4 HX711, U5 TMC6300, U6 AP2114HA-3.3, U7 SN74LV1T34DBV, U8 VEML7700, U9 TS1117BCW33_RPG

Commit message: Mod v1
- ESP32-S3-MINI-1N8
- 24x WS2812 20x20 LED
- SMD Resistors 4 direction Force Sensor
- Accelerometer
Parts:
- removed C11: 0.1uF, Capacitor_SMD:C_0603_1608Metric, symbol Device:C_Small
- removed J4: A, SolderPads:SolderPads_2mm_3_STRAIN, symbol Connector_Generic:Conn_01x03
- removed J5: B, SolderPads:SolderPads_2mm_3_STRAIN, symbol Connector_Generic:Conn_01x03
- removed NT1: NetTie_2, NetTie:NetTie-2_SMD_Pad0.5mm, symbol Device:NetTie_2
- removed Q2: UMH3N, Package_TO_SOT_SMD:SOT-363_SC-70-6, symbol Transistor_BJT:UMH3N
- removed TP13: EN, Modified:TestPoint_Pad_D2.0mm_ValueSilk, symbol Connector:TestPoint_Small
- removed TP14: BOOT, Modified:TestPoint_Pad_D2.0mm_ValueSilk, symbol Connector:TestPoint_Small
- removed TP15: TX, Modified:TestPoint_Pad_D2.0mm_ValueSilk, symbol Connector:TestPoint_Small
- removed TP16: RX, Modified:TestPoint_Pad_D2.0mm_ValueSilk, symbol Connector:TestPoint_Small
- removed U2: T-Micro32_Plus, lilygo_micro32:T-Micro32, symbol lilygo_micro32:T-Micro32_Plus
- removed U3: CH340C, Package_SO:SOIC-16_3.9x9.9mm_P1.27mm, symbol Interface_USB:CH340C
- removed U9: TS1117BCW33_RPG, Package_TO_SOT_SMD:SOT-223-3_TabPin2, symbol Regulator_Linear:TS1117BCW33_RPG
- removed Z1, Z2, Z3, Z4: BF350-3AA Strain Gauge, strain:BF350-3AA, symbol no_pin:no_pin
- removed Z5: dummy_keepouts, view_custom:ViewKeepouts3d, symbol no_pin:no_pin
- added C12, C17, C5: 10uF, Capacitor_SMD_AKL:C_0805_2012Metric, symbol Device:C_Small
- added C13, C18, C20, C23, C37, C38, C39, C40, C41, C42, C43, C44, C45, C46, C47, C48, C49, C50, C51, C52, C6: 0.1uF, Capacitor_SMD_AKL:C_0603_1608Metric, symbol Device:C_Small
- added C53: 1uF, Capacitor_SMD_AKL:C_0603_1608Metric, symbol Device:C_Small
- added D10, D11, D12, D13, D14, D15, D16, D17, D18, D19, D20, D21, D22, D23, D24, D9: WS2812-2020, CrumpPrints:WS2812-2020, symbol crumpschemes:WS2812-2020
- added IC1: MXC6655XA, MXC6655XA, symbol MXC6655XA:MXC6655XA
- added L2: 3.3uH, Inductor_SMD_AKL:L_0805_2012Metric, symbol Device:L_Small
- added Q2: MMBT4403, Package_TO_SOT_SMD_AKL:SOT-23, symbol Device:Q_PNP_BEC
- added R15: 10k, Resistor_SMD_AKL:R_0603_1608Metric, symbol Device:R_Small
- added R17: 8.2k, Resistor_SMD_AKL:R_0603_1608Metric, symbol Device:R_Small
- added R19, R20, R21, R23, R24, R25: 100, Resistor_SMD_AKL:R_0603_1608Metric, symbol Device:R_Small
- added R26, R27, R28, R29, R30, R32, R34, R36: 1K, Resistor_SMD_AKL:R_2512_6332Metric, symbol Device:R_Small
- added R31, R33, R35, R37, R38, R39, R40, R41: 1k, Resistor_SMD_AKL:R_0603_1608Metric, symbol Device:R_Small
- added R42, R44: 2.7k, Resistor_SMD_AKL:R_0603_1608Metric, symbol Device:R_Small
- added TP3: TX, Modified:TestPoint_Pad_D2.0mm_ValueSilk, symbol Connector:TestPoint_Small
- added TP4: RX, Modified:TestPoint_Pad_D2.0mm_ValueSilk, symbol Connector:TestPoint_Small
- added U2: ESP32-S3-MINI-1, Espressif:ESP32-S3-MINI-1, symbol ESP:ESP32-S3-MINI-1
- added U4: HX711, Package_SO_AKL:SOIC-16_3.9x9.9mm_P1.27mm, symbol strain:HX711
- added Z6: dummy_keepouts, view_custom:ViewKeepouts3d, symbol no_pin:no_pin
- C1: renamed from C9; footprint Capacitor_SMD:C_0805_2012Metric -> Capacitor_SMD_AKL:C_0805_2012Metric
- C10: renamed from C16; footprint Capacitor_SMD:C_0805_2012Metric -> Capacitor_SMD_AKL:C_0805_2012Metric
- C11: renamed from C12; footprint Capacitor_SMD:C_0603_1608Metric -> Capacitor_SMD_AKL:C_0603_1608Metric
- C14: renamed from C27; footprint Capacitor_SMD:C_0603_1608Metric -> Capacitor_SMD_AKL:C_0603_1608Metric
- C15: renamed from C18; footprint Capacitor_SMD:C_0805_2012Metric -> Capacitor_SMD_AKL:C_0805_2012Metric
- C16: renamed from C19; footprint Capacitor_SMD:C_0603_1608Metric -> Capacitor_SMD_AKL:C_0603_1608Metric
- C19: renamed from C22; footprint Capacitor_SMD:C_0603_1608Metric -> Capacitor_SMD_AKL:C_0603_1608Metric
- C2: renamed from C10; footprint Capacitor_SMD:C_0805_2012Metric -> Capacitor_SMD_AKL:C_0805_2012Metric
- C21: renamed from C17; footprint Capacitor_SMD:C_0603_1608Metric -> Capacitor_SMD_AKL:C_0603_1608Metric
- C22: renamed from C23; footprint Capacitor_SMD:C_0603_1608Metric -> Capacitor_SMD_AKL:C_0603_1608Metric
- C24: value 10uF -> 0.1uF; footprint Capacitor_SMD:C_0805_2012Metric -> Capacitor_SMD_AKL:C_0603_1608Metric; Digikey 1276-2891-1-ND -> 1276-1935-1-ND; LCSC C2922480 -> C1591; Mouser 187-CL21A106KAYNNNE -> 187-CL10B104KB8NNWC
- C25: footprint Capacitor_SMD:C_0603_1608Metric -> Capacitor_SMD_AKL:C_0603_1608Metric
- C26: renamed from C21; footprint Capacitor_SMD:C_0603_1608Metric -> Capacitor_SMD_AKL:C_0603_1608Metric
- C27: renamed from C29; footprint Capacitor_SMD:C_0603_1608Metric -> Capacitor_SMD_AKL:C_0603_1608Metric
- C28: renamed from C20; footprint Capacitor_SMD:C_0603_1608Metric -> Capacitor_SMD_AKL:C_0603_1608Metric
- C29: renamed from C1; footprint Capacitor_SMD:C_0603_1608Metric -> Capacitor_SMD_AKL:C_0603_1608Metric
- C3: renamed from C26; footprint Capacitor_SMD:C_0805_2012Metric -> Capacitor_SMD_AKL:C_0805_2012Metric
- C30: renamed from C2; footprint Capacitor_SMD:C_0603_1608Metric -> Capacitor_SMD_AKL:C_0603_1608Metric
- C31: renamed from C3; footprint Capacitor_SMD:C_0603_1608Metric -> Capacitor_SMD_AKL:C_0603_1608Metric
- C32: renamed from C4; footprint Capacitor_SMD:C_0603_1608Metric -> Capacitor_SMD_AKL:C_0603_1608Metric
- C33: renamed from C5; footprint Capacitor_SMD:C_0603_1608Metric -> Capacitor_SMD_AKL:C_0603_1608Metric
- C34: renamed from C6; footprint Capacitor_SMD:C_0603_1608Metric -> Capacitor_SMD_AKL:C_0603_1608Metric
- C35: renamed from C7; footprint Capacitor_SMD:C_0603_1608Metric -> Capacitor_SMD_AKL:C_0603_1608Metric
- C36: renamed from C8; footprint Capacitor_SMD:C_0603_1608Metric -> Capacitor_SMD_AKL:C_0603_1608Metric
- C4: renamed from C28; footprint Capacitor_SMD:C_0603_1608Metric -> Capacitor_SMD_AKL:C_0603_1608Metric
- C7: renamed from C13; footprint Capacitor_SMD:C_0805_2012Metric -> Capacitor_SMD_AKL:C_0805_2012Metric
- C8: renamed from C14; footprint Capacitor_SMD:C_0603_1608Metric -> Capacitor_SMD_AKL:C_0603_1608Metric
- C9: renamed from C15; footprint Capacitor_SMD:C_0603_1608Metric -> Capacitor_SMD_AKL:C_0603_1608Metric
- D1, D2, D3, D4, D5, D6, D7, D8: value SK6812SIDE-A -> WS2812-2020; footprint sk6812:SK6812-SIDE-A -> CrumpPrints:WS2812-2020; symbol SK6812:SK6812SIDE-A -> crumpschemes:WS2812-2020
- L1: footprint Inductor_SMD:L_0805_2012Metric -> Inductor_SMD_AKL:L_0805_2012Metric
- Q1: footprint Package_TO_SOT_SMD:SOT-23 -> Package_TO_SOT_SMD_AKL:SOT-23
- R1: renamed from R7; footprint Resistor_SMD:R_0603_1608Metric -> Resistor_SMD_AKL:R_0603_1608Metric
- R10: renamed from R2; footprint Resistor_SMD:R_0603_1608Metric -> Resistor_SMD_AKL:R_0603_1608Metric
- R11, R12: footprint Resistor_SMD:R_0603_1608Metric -> Resistor_SMD_AKL:R_0603_1608Metric
- R13: renamed from R14; footprint Resistor_SMD:R_0603_1608Metric -> Resistor_SMD_AKL:R_0603_1608Metric
- R14: renamed from R3; footprint Resistor_SMD:R_0603_1608Metric -> Resistor_SMD_AKL:R_0603_1608Metric
- R16: renamed from R4; footprint Resistor_SMD:R_0603_1608Metric -> Resistor_SMD_AKL:R_0603_1608Metric
- R18: renamed from R5; footprint Resistor_SMD:R_0603_1608Metric -> Resistor_SMD_AKL:R_0603_1608Metric
- R2: renamed from R8; footprint Resistor_SMD:R_0603_1608Metric -> Resistor_SMD_AKL:R_0603_1608Metric
- R22: renamed from R6; footprint Resistor_SMD:R_0603_1608Metric -> Resistor_SMD_AKL:R_0603_1608Metric
- R3: renamed from R9; footprint Resistor_SMD:R_0603_1608Metric -> Resistor_SMD_AKL:R_0603_1608Metric
- R4: renamed from R17; footprint Resistor_SMD:R_0603_1608Metric -> Resistor_SMD_AKL:R_0603_1608Metric
- R5: renamed from R1; footprint Resistor_SMD:R_0603_1608Metric -> Resistor_SMD_AKL:R_0603_1608Metric
- R6: renamed from R15; footprint Resistor_SMD:R_0603_1608Metric -> Resistor_SMD_AKL:R_0603_1608Metric
- R7: renamed from R16; footprint Resistor_SMD:R_0603_1608Metric -> Resistor_SMD_AKL:R_0603_1608Metric
- R8: renamed from R13; footprint Resistor_SMD:R_0603_1608Metric -> Resistor_SMD_AKL:R_0603_1608Metric
- R9: renamed from R10; footprint Resistor_SMD:R_0603_1608Metric -> Resistor_SMD_AKL:R_0603_1608Metric
- U1: renamed from U6; footprint Package_TO_SOT_SMD:SOT-223-3_TabPin2 -> Package_TO_SOT_SMD_AKL:SOT-223-3_TabPin2; Digikey AP2114HA-3.3TRG1DICT-ND, or MIC39100-3.3WS-CT-ND -> AP2114HA-3.3TRG1DICT-ND; Note Populate either U6 or U9 - depending on pinout - but not bo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 -> (none)
- U3: renamed from U4; footprint Package_SO:SOIC-16_3.9x9.9mm_P1.27mm -> Package_SO_AKL:SOIC-16_3.9x9.9mm_P1.27mm
- U7: renamed from U1; footprint Package_SO:SOIC-8_3.9x4.9mm_P1.27mm -> Package_SO_AKL:SOIC-8_3.9x4.9mm_P1.27mm; LCSC C2856764, or C3003196 -> C2856764
- U8: renamed from U7; footprint Package_TO_SOT_SMD:SOT-23-5 -> Package_TO_SOT_SMD_AKL:SOT-23-5
- Z5: renamed from Z10; AliExpress (none) -> https://www.aliexpress.com/item/1005001384349991.html; Note SparkFun: https://www.sparkfun.com/products/20441 -> (none)
- renumbered J3 to J1, J1 to J3, TP8 to TP10, TP12 to TP11, TP9 to TP12, TP10 to TP13, TP11 to TP14, TP3 to TP5, TP4 to TP6, TP5 to TP7, TP6 to TP8, TP7 to TP9, U8 to U6, Z6 to Z1, Z7 to Z2, Z8 to Z3, Z9 to Z4
Connections:
- net LCD_BACKLIGHT is gone; now on net LCD_SCK: J1.6 (Pin_6)
- net +3V3: now also C28.2, J1.2 (Pin_2), C12.1, C13.1, C5.1, C53.2, C6.1, IC1.7 (VDD), Q2.2 (E), U2.3 (3V3), U4.1 (VSUP), U4.15 (RATE), U4.16 (DVDD); no longer C24.1, C25.1, C28.1, J1.1 (Pin_1)
- net +5V: now also D1.4 (VDD), D2.4 (VDD), D3.4 (VDD), D4.4 (VDD), D5.4 (VDD), D6.4 (VDD), D7.4 (VDD), D8.4 (VDD), C37.1, C38.1, C39.1, C40.1, C41.1, C42.1, C43.1, C44.1, C45.1, C46.1, C47.1, C48.1, C49.1, C50.1, C51.1, C52.1, D10.4 (VDD), D11.4 (VDD), D12.4 (VDD), D13.4 (VDD), D14.4 (VDD), D15.4 (VDD), D16.4 (VDD), D17.4 (VDD), D18.4 (VDD), D19.4 (VDD), D20.4 (VDD), D21.4 (VDD), D22.4 (VDD), D23.4 (VDD), D24.4 (VDD), D9.4 (VDD); no longer D1.2 (VDD), D2.2 (VDD), D3.2 (VDD), D4.2 (VDD), D5.2 (VDD), D6.2 (VDD), D7.2 (VDD), D8.2 (VDD)
- net ESP32_EN: now also U2.45 (EN)
- net GND: now also C10.2, C11.2, C15.2, C16.2, C19.1, C28.1, D1.2 (VSS), D2.2 (VSS), D3.2 (VSS), D4.2 (VSS), D5.2 (VSS), D6.2 (VSS), D7.2 (VSS), D8.2 (VSS), J1.1 (Pin_1), R16.2, U3.14 (XI), U3.5 (AGND), C12.2, C13.2, C17.2, C18.2, C20.1, C37.2, C38.2, C39.2, C40.2, C41.2, C42.2, C43.2, C44.2, C45.2, C46.2, C47.2, C48.2, C49.2, C5.2, C50.2, C51.2, C52.2, C53.1, C6.2, D10.2 (VSS), D11.2 (VSS), D12.2 (VSS), D13.2 (VSS), D14.2 (VSS), D15.2 (VSS), D16.2 (VSS), D17.2 (VSS), D18.2 (VSS), D19.2 (VSS), D20.2 (VSS), D21.2 (VSS), D22.2 (VSS), D23.2 (VSS), D24.2 (VSS), D9.2 (VSS), IC1.9 (GND), R17.2, R30.2, R32.2, R34.2, R36.2, R38.2, R39.2, R40.2, R41.2, U2.1 (GND), U2.2 (GND), U2.42 (GND), U2.43 (GND), U2.46 (GND), U4.14 (XI), U4.5 (AGND); no longer C24.2, C25.2, C28.2, D1.4 (VSS), D2.4 (VSS), D3.4 (VSS), D4.4 (VSS), D5.4 (VSS), D6.4 (VSS), D7.4 (VSS), D8.4 (VSS), J1.2 (Pin_2)
- net LCD_CMD: now also J1.4 (Pin_4), U2.20 (GPIO16/U0CTS/ADC2_CH5/XTAL_32K_NH5); no longer J1.8 (Pin_8)
- net LCD_CS: now also J1.5 (Pin_5), U2.19 (GPIO15/U0RTS/ADC2_CH4/XTAL_32K_P); no longer J1.7 (Pin_7)
- net LCD_DATA: now also J1.7 (Pin_7), U2.17 (GPIO13/TOUCH13/ADC2_CH2/FSPIQ/FSPIIO7/SUBSPIQ); no longer J1.5 (Pin_5)
- net LCD_RST: now also J1.8 (Pin_8), U2.16 (GPIO12/TOUCH11/ADC2_CH0/FSPICS0/FSPIIO4/SUBSPICS0); no longer J1.3 (Pin_3)
- net LCD_SCK: now also U2.18 (GPIO14/TOUCH14/ADC2_CH3/FSPIWP/FSPIDQS/SUBSPIWP); no longer J1.4 (Pin_4)
- net LED_DATA_5V: now also D1.3 (DIN); no longer D1.1 (DIN)
- net MAG_CLK: now also U2.26 (GPIO26)
- net MAG_CSN: now also U2.25 (GPIO21)
- net MAG_DO: now also U2.27 (GPIO47/SPICLK_P/SUBSPICLK_P_DIFF)
- net SCL: now also R42.1, U2.28 (SPIIO4/GPIO33/FSPIHD/SUBSPIHD)
- net SDA: now also R44.2, U2.29 (SPIIO5/GPIO34/FSPICS0/SUBSPICS0)
- net TMC_DIAG: now also U2.12 (GPIO8/TOUCH8/ADC1_CH7/SUBSPICS1)
- net TMC_UH: now also U2.5 (GPIO1/TOUCH1/ADC1_CH0)
- net TMC_UL: now also U2.9 (GPIO5/TOUCH5/ADC1_CH4)
- net TMC_VH: now also U2.6 (GPIO2/TOUCH2/ADC1_CH1)
- net TMC_VL: now also U2.11 (GPIO7/TOUCH7/ADC1_CH6)
- net TMC_WH: now also U2.8 (GPIO4/TOUCH4/ADC1_CH3)
- net TMC_WL: now also U2.10 (GPIO6/TOUCH6/ADC1_CH5)
- net USB_D+: now also U2.24 (GPIO20/U1CTS/ADC2_CH9/CLK_OUT1/USB_D+)
- net USB_D-: now also U2.23 (GPIO19/U1RTS/ADC2_CH8/CLK_OUT2/USB_D-)
- net at D2.1 (DOUT): now also D3.3 (DIN); no longer D1.3 (DOUT)
- net at D2.3 (DIN): now also D1.1 (DOUT); no longer D3.1 (DIN)
- net at D4.1 (DOUT): now also D5.3 (DIN); no longer D3.3 (DOUT)
- net at D4.3 (DIN): now also D3.1 (DOUT); no longer D5.1 (DIN)
- net at D6.1 (DOUT): now also D7.3 (DIN); no longer D5.3 (DOUT)
- net at D6.3 (DIN): now also D5.1 (DOUT); no longer D7.1 (DIN)
- net at D8.1 (DOUT): now also D9.3 (DIN); no longer D7.3 (DOUT)
- net at D8.3 (DIN): now also D7.1 (DOUT)
- removed net GNDA: C10.2, C11.2, C15.2, C16.2, C19.1, R16.2, U3.10 (INB+), U3.14 (XI), U3.5 (AGND), U3.9 (INB-)
- net LED_DATA_3V3 renamed LED_DATA
- net LED_DATA: now also U2.30 (GPIO48/SPICLK_N/SUBSPICLK_N_DIFF)
- net STRAIN_DO renamed STRAIN1_DO
- net STRAIN1_DO: now also U2.33 (SPIDQS/GPIO37/FSPIQ/SUBSPIQ)
- net STRAIN_E+ renamed AVDD
- net AVDD: now also C17.1, C18.1, L2.2, R26.2, R27.2, R28.2, R29.2, R31.1, R33.1, R35.1, R37.1
- net STRAIN_S+ renamed IN1A+
- net IN1A+: now also R26.1, R30.1
- net STRAIN_S- renamed IN1A-
- net IN1A-: now also R31.2, R38.1
- net STRAIN_SCK renamed STRAIN1_SCK
- net STRAIN1_SCK: now also U2.34 (GPIO38/FSPIWP/SUBSPIWP)
- new net: C23.1, R19.2, U3.10 (INB+)
- new net: C23.2, R23.1, U3.9 (INB-)
- new net: D10.1 (DOUT), D11.3 (DIN)
- new net: D10.3 (DIN), D9.1 (DOUT)
- new net: D13.1 (DOUT), D14.3 (DIN)
- new net: D12.1 (DOUT), D13.3 (DIN)
- new net: R15.2, R17.1, U4.4 (VFB)
- new net: IC1.12 (SCL), R42.2
- new net: C24.2, R20.1, U4.7 (INA-)
- new net: TP3.1, U2.39 (U0TXD/GPIO43/CLK_OUT1)
- new net: D11.1 (DOUT), D12.3 (DIN)
- new net: D20.1 (DOUT), D21.3 (DIN)
- new net: D19.1 (DOUT), D20.3 (DIN)
- new net: D14.1 (DOUT), D15.3 (DIN)
- new net: D21.1 (DOUT), D22.3 (DIN)
- new net: D22.1 (DOUT), D23.3 (DIN)
- new net: C25.1, R21.2, U4.10 (INB+)
- new net: C25.2, R25.1, U4.9 (INB-)
- new net: C24.1, R24.2, U4.8 (INA+)
- new net: D15.1 (DOUT), D16.3 (DIN)
- new net: IC1.2 (SDA), R44.1
- new net: D17.1 (DOUT), D18.3 (DIN)
- new net: D16.1 (DOUT), D17.3 (DIN)
- new net: TP4.1, U2.40 (U0RXD/GPIO44/CLK_OUT2)
- new net: D23.1 (DOUT), D24.3 (DIN)
- new net: L2.1, Q2.3 (C), R15.1, U4.3 (AVDD)
- new net: D18.1 (DOUT), D19.3 (DIN)
- new net: C20.2, U4.6 (VBG)
- new net: Q2.1 (B), U4.2 (BASE)
- new net IN1B+: R19.1, R27.1, R32.1
- new net IN1B-: R23.2, R33.2, R39.1
- new net IN2A+: R24.1, R28.1, R34.1
- new net IN2A-: R20.2, R35.2, R40.1
- new net IN2B+: R21.1, R29.1, R36.1
- new net IN2B-: R25.2, R37.2, R41.1
- new net LCD_BL: J1.3 (Pin_3), U2.21 (GPIO17/U1TXD/ADC2_CH6)
- new net STRAIN2_DO: U2.31 (SPIIO6/GPIO35/FSPID/SUBSPID), U4.12 (DOUT)
- new net STRAIN2_SCK: U2.32 (SPIIO7/GPIO36/FSPICLK/SUBSPICLK), U4.11 (PD_SCK)
- no-connect marks 24 -> 36
Other:
- note added: "Accelerometer"
- note added: "LEDS - BOOSTER"
- note added: "MCU - ESP32-S3"
- note removed: "GPIO12=MTDI. Should be 0 on boot for 3.3v built-in flash/psram on ESP32-PICO-v3-02"
- note removed: "IO2 must be 0 to enter UART download mode"
- note removed: "If your voltage regulator follows the 5V-GND-3V3 pinout (AP2114HA) populate your regulator on the footprint labled U6. If your regulator follows the pinout of GND-3V3-5V (TS1117BCW33) populate your regulator on the footprint labaled U9)."
- note removed: "MCU - ESP32 (T-MICRO32 PLUS)"
- note removed: "Rate=1 --> 80 samples per second"
- note removed: "Reset/Boot via USB serial"
- note removed: "Use either U6 or U9, but not both!"
- moved on the sheet: C1, C10, C11, C14, C15, C16, C19, C2, C21, C22, C26, C27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
